File: docs/Schematics/DummyLoad/DummyLoad.kicad_pcb (KiCad board)
At the start: 4 copper layers, 218 x 230 mm, 83 parts, among them J1 Conn_Coaxial, J2 Conn_Coaxial, J3 Fan, J4 PSU, J5 AMP_left, J6 AMP_right, J7 MCU, K1 J123F1C12VDC.36, K2 J123F1C12VDC.36, K3 J123F1C12VDC.36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

Commit message: Version 1.0 of the audio analyzer and fix embedded repo warnings
Other:
- board text added: "Astatine - DummyLoad 4/8Ω V1.0"
- board text added: "Left Channel"
- board text added: "Right Channel"
